File: KiCad/ardInclinometer-ATmega328/ATmega328.kicad_sch (KiCad schematic)
At the start: 11 parts, among them J2 Power in, J3 FTDI, U2 AMS1117-5.0, U3 ATmega328P-PU, Y1 16MHz

Commit message: new schematics and pcb
Parts:
- renumbered J2 to J1, J3 to J2, U2 to U3, U3 to U4
Connections:
- net A4 renamed A4/SDA
- net A5 renamed A5/SCL
Changed lines of the file:
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@@
     (title "ardInclinometer-ATmega328")
     (date "2022-09-09")
-    (rev "0.1")
+    (rev "0.2")
   )
   (junction (at 220.98 134.62) (diameter 0) (color 0 0 0 0)
@@
     )
   )
-  (global_label "A5" (shape input) (at 175.26 93.98 0) (fields_autoplaced)
-    (effects (font (size 1.27 1.27)) (justify left))
-    (property "Intersheet References" "${INTERSHEET_REFS}" (id 0) (at 179.9712 93.9006 0)
+  (global_label "A5{slash}SCL" (shape input) (at 175.26 93.98 0) (fields_autoplaced)
+    (effects (font (size 1.27 1.27)) (justify left))
+    (property "Intersheet References" "${INTERSHEET_REFS}" (id 0) (at 184.8093 93.9006 0)
       (effects (font (size 1.27 1.27)) (justify left) hide)
     )
@@
     )
   )
-  (global_label "A4" (shape input) (at 162.56 91.44 0) (fields_autoplaced)
-    (effects (font (size 1.27 1.27)) (justify left))
-    (property "Intersheet References" "${INTERSHEET_REFS}" (id 0) (at 167.2712 91.3606 0)
+  (global_label "A4{slash}SDA" (shape input) (at 162.56 91.44 0) (fields_autoplaced)
+    (effects (font (size 1.27 1.27)) (justify left))
+    (property "Intersheet References" "${INTERSHEET_REFS}" (id 0) (at 172.1698 91.3606 0)
       (effects (font (size 1.27 1.27)) (justify left) hide)
     )
@@
   (symbol (lib_id "My_Misc:ATmega328P-PU") (at 142.24 88.9 0) (unit 1)
     (in_bom yes) (on_board yes) (fields_autoplaced)
-    (property "Reference" "U3" (id 0) (at 119.38 54.0893 0))
+    (property "Reference" "U4" (id 0) (at 119.38 54.0893 0))
     (property "Value" "ATmega328P-PU" (id 1) (at 119.38 56.6293 0))
     (property "Footprint" "My_Misc:DIP-28_W7.62mm_LongPads w socket" (id 2) (at 142.24 88.9 0)
@@
   (symbol (lib_id "Regulator_Linear:AMS1117-5.0") (at 63.5 92.71 0) (unit 1)
     (in_bom yes) (on_board yes) (fields_autoplaced)
-    (property "Reference" "U2" (id 0) (at 63.5 85.09 0))
+    (property "Reference" "U3" (id 0) (at 63.5 85.09 0))
     (property "Value" "AMS1117-5.0" (id 1) (at 63.5 87.63 0))
     (property "Footprint" "Package_TO_SOT_SMD:SOT-223-3_TabPin2" (id 2) (at 63.5 87.63 0)
@@
   (symbol (lib_id "My_Headers:6-pin_FTDI_header") (at 210.82 50.8 0) (unit 1)
     (in_bom yes) (on_board yes) (fields_autoplaced)
-    (property "Reference" "J3" (id 0) (at 211.455 40.64 0))
+    (property "Reference" "J2" (id 0) (at 211.455 40.64 0))
     (property "Value" "FTDI" (id 1) (at 211.455 43.18 0))
     (property "Footprint" "My_Headers:6-pin FTDI Programmer PinSocket large" (id 2) (at 210.82 50.8 0)
@@
   (symbol (lib_id "My_Headers:2-pin_power_input_header") (at 60.96 45.72 0) (unit 1)
     (in_bom yes) (on_board yes) (fields_autoplaced)
-    (property "Reference" "J2" (id 0) (at 62.23 46.9899 0)
+    (property "Reference" "J1" (id 0) (at 62.23 46.9899 0)
       (effects (font (size 1.27 1.27)) (justify left))
     )

Commit message: more mistakes corrected...
Parts:
- added JP1: Power from FTDI, My_Parts:Jumper_1x02_P2.54mm_large, symbol Jumper:Jumper_2_Open
Connections:
- net +5V: now also JP1.2 (B); no longer J2.3 (VCC)
- new net: J2.3 (VCC), JP1.1 (A)
Changed lines of the file:
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@@
     (title "ardInclinometer-ATmega328")
     (date "2022-09-09")
-    (rev "0.2")
+    (rev "0.4")
   )
   (junction (at 220.98 134.62) (diameter 0) (color 0 0 0 0)
@@
   (junction (at 142.24 132.08) (diameter 0) (color 0 0 0 0)
   )
+  (wire (pts (xy 226.06 29.21) (xy 226.06 34.29))
+    (stroke (width 0) (type default) (color 0 0 0 0))
+  )
   (wire (pts (xy 63.5 110.49) (xy 50.8 110.49))
     (stroke (width 0) (type default) (color 0 0 0 0))
@@
     (stroke (width 0) (type default) (color 0 0 0 0))
   )
+  (wire (pts (xy 226.06 44.45) (xy 226.06 50.8))
+    (stroke (width 0) (type default) (color 0 0 0 0))
+  )
   (wire (pts (xy 50.8 110.49) (xy 50.8 105.41))
     (stroke (width 0) (type default) (color 0 0 0 0))
@@
   )
   (wire (pts (xy 71.12 92.71) (xy 76.2 92.71))
-    (stroke (width 0) (type default) (color 0 0 0 0))
-  )
-  (wire (pts (xy 226.06 50.8) (xy 226.06 40.64))
     (stroke (width 0) (type default) (color 0 0 0 0))
   )
@@
     (pin "2")
   )
-  (symbol (lib_id "power:+5V") (at 226.06 40.64 0) (unit 1)
-    (in_bom yes) (on_board yes) (fields_autoplaced)
-    (property "Reference" "#PWR018" (id 0) (at 226.06 44.45 0)
-      (effects (font (size 1.27 1.27)) hide)
-    )
-    (property "Value" "+5V" (id 1) (at 226.06 35.56 0))
-    (property "Footprint" "" (id 2) (at 226.06 40.64 0)
-      (effects (font (size 1.27 1.27)) hide)
-    )
-    (property "Datasheet" "" (id 3) (at 226.06 40.64 0)
+  (symbol (lib_id "power:+5V") (at 226.06 29.21 0) (unit 1)
+    (in_bom yes) (on_board yes) (fields_autoplaced)
+    (property "Reference" "#PWR018" (id 0) (at 226.06 33.02 0)
+      (effects (font (size 1.27 1.27)) hide)
+    )
+    (property "Value" "+5V" (id 1) (at 226.06 24.13 0))
+    (property "Footprint" "" (id 2) (at 226.06 29.21 0)
+      (effects (font (size 1.27 1.27)) hide)
+    )
+    (property "Datasheet" "" (id 3) (at 226.06 29.21 0)
       (effects (font (size 1.27 1.27)) hide)
     )
@@
     (pin "1")
   )
+  (symbol (lib_id "Jumper:Jumper_2_Open") (at 226.06 39.37 90) (unit 1)
+    (in_bom yes) (on_board yes) (fields_autoplaced)
+    (property "Reference" "JP1" (id 0) (at 227.33 38.0999 90)
+      (effects (font (size 1.27 1.27)) (justify right))
+    )
+    (property "Value" "Power from FTDI" (id 1) (at 227.33 40.6399 90)
+      (effects (font (size 1.27 1.27)) (justify right))
+    )
+    (property "Footprint" "My_Parts:Jumper_1x02_P2.54mm_large" (id 2) (at 226.06 39.37 0)
+      (effects (font (size 1.27 1.27)) hide)
+    )
+    (property "Datasheet" "~" (id 3) (at 226.06 39.37 0)
+      (effects (font (size 1.27 1.27)) hide)
+    )
+    (pin "1")
+    (pin "2")
+  )
   (symbol (lib_id "power:VCC") (at 50.8 83.82 0) (unit 1)

Commit message: kicad corrections and dev
Parts:
- added C3, C4: 100n, My_Misc:C_Disc_D4.3mm_W1.9mm_P5.00mm_large, symbol Device:C
- C7: renamed from C5; footprint My_Misc:C_Disc_D3.0mm_W1.6mm_P2.50mm_larg -> My_Misc:C_Disc_D4.3mm_W1.9mm_P5.00mm_large
- renumbered C3 to C5, C4 to C6, R11 to R13
Connections:
- net +5V: now also C3.1, C4.2
- net GND: now also C3.2, C4.1
- net AREF: now reaches U4.21 (AREF)
- net D11 renamed D11/MOSI
- net D12 renamed D12/MISO
- net D13 renamed D13/SCK
