File: KiCad/ardInclinometer-ATmega328/ardInclinometer-ATmega328.kicad_pcb (KiCad board)
At the start: 2 copper layers, 66.7 x 55.9 mm, 37 parts, among them J1 1.8" display, J2 Power in, J3 FTDI, SW1 Lock X, SW2 Lock Y, SW3 Lock Z, SW4 Lock all, SW5 SW_Push, U1 GY-521_MPU-6050, U2 AMS1117-5.0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

Commit message: new schematics and pcb
Parts:
- removed the J1 at (186.1, 71.3)
- added JP1: FTDI power, My_Parts:Jumper_1x02_P2.54mm_large, B.Cu at (169.9, 66.5)
- added U2: SSD1306_I2C_display, My_Parts:SSD1306_I2C_0.96_OLED_display_large, F.Cu at (185.9, 71.5)
- moved C1 4.73 mm to (177.9, 78.5)
- moved J1 4.42 mm to (179.5, 83.5)
- renumbered J2 to J1, J3 to J2, U2 to U3, U3 to U4
Connections:
- net A4 renamed A4/SDA
- net A5 renamed A5/SCL
- U1 pad 1: +5V -> Net-(U1-Pad1)
Routing:
- net Net-(U1-Pad1): track 0.00 -> 67.7 mm
- net A5/SCL: track 73.1 -> 61.0 mm
- net GND: track 191.7 -> 182.6 mm
- net D6: track 67.1 -> 58.4 mm
- net +5V: track 200.1 -> 191.9 mm, vias 1 -> 0
- net VCC: track 10.1 -> 16.2 mm
- net D10: track 36.1 -> 30.2 mm
- net D13: track 35.0 -> 29.9 mm
- net D9: track 28.2 -> 33.1 mm
- net D12: track 32.8 -> 30.2 mm
- net D5: track 65.4 -> 63.5 mm
- net D4: track 64.8 -> 66.0 mm
- net A4/SDA: track 71.5 -> 70.5 mm
- net D3: track 75.5 -> 76.1 mm
- net D2: track 64.4 -> 64.9 mm

Commit message: more mistakes corrected...
Parts:
- JP1: value FTDI power -> Power from FTDI
- moved JP1 3.61 mm to (166.9, 64.5), turned to -90 degrees
Connections:
- J2 pad 3: +5V -> Net-(J2-Pad3)
- JP1 pad 1: Net-(U1-Pad1) -> Net-(J2-Pad3)
- U1 pad 1: Net-(U1-Pad1) -> +5V
Routing:
- net Net-(U1-Pad1): track 67.7 -> 0.00 mm
- net +5V: track 191.9 -> 209.8 mm
- net Net-(J2-Pad3): track 0.00 -> 15.2 mm
- net D2: track 64.9 -> 79.9 mm
- net GND: track 182.6 -> 191.3 mm
- net D10: track 30.2 -> 37.6 mm
- net A5/SCL: track 61.0 -> 66.6 mm
- net D6: track 58.4 -> 62.4 mm
- net A4/SDA: track 70.5 -> 66.8 mm
- net D9: track 33.1 -> 30.7 mm
- net D5: track 63.5 -> 65.4 mm
- net D13: track 29.9 -> 31.8 mm
- net D3: track 76.1 -> 74.3 mm
- net D12: track 30.2 -> 28.4 mm
- removed copper zone on B.Cu, net GND

Commit message: kicad corrections and dev
Parts:
- added C3: 100n, My_Misc:C_Disc_D4.3mm_W1.9mm_P5.00mm_large, F.Cu at (158.9, 83.0)
- added C4: 100n, My_Misc:C_Disc_D4.3mm_W1.9mm_P5.00mm_large, F.Cu at (174.9, 90.5)
- added R11: 4.7k, My_Misc:R_Axial_DIN0207_L6.3mm_D2.5mm_P10.16mm_Horizontal_large, F.Cu at (209.9, 114.5)
- added R12: 4.7k, My_Misc:R_Axial_DIN0207_L6.3mm_D2.5mm_P10.16mm_Horizontal_large, F.Cu at (170.9, 114.5)
- C7: renamed from C5; footprint My_Misc:C_Disc_D3.0mm_W1.6mm_P2.50mm_larg -> My_Misc:C_Disc_D4.3mm_W1.9mm_P5.00mm_large
- J1: moved to B.Cu
- moved C7 45.1 mm to (194.9, 63.5), turned to -90 degrees
- moved C1 34.2 mm to (209.9, 66.5)
- moved J2 30.6 mm to (189.6, 66.5), turned to 90 degrees
- moved J1 26.3 mm to (199.9, 67.0), turned to 0 degrees
- moved C2 18.6 mm to (189.9, 80.5)
- moved U3 8.08 mm to (197.9, 78.5)
- moved JP1 3.16 mm to (169.9, 65.5), turned to 90 degrees
- renumbered C3 to C5, C4 to C6, R11 to R13
Connections:
- net D11 renamed D11/MOSI
- net D12 renamed D12/MISO
- net D13 renamed D13/SCK
- U4 pad 21: unconnected-(U4-Pad21) -> AREF
Routing:
- net +5V: track 209.8 -> 263.3 mm
- net GND: track 191.3 -> 214.0 mm
- net D0/Rx: track 4.39 -> 23.1 mm
- net D1/Tx: track 4.39 -> 22.6 mm
- net Net-(C7-Pad1): track 5.07 -> 19.3 mm
- net A4/SDA: track 66.8 -> 79.2 mm
- net A5/SCL: track 66.6 -> 77.2 mm
- net D10: track 37.6 -> 30.5 mm
- net D2: track 79.9 -> 73.1 mm
- net VCC: track 16.2 -> 20.4 mm
- net D6: track 62.4 -> 58.2 mm
- net D3: track 74.3 -> 75.5 mm
- net D9: track 30.7 -> 31.8 mm
- net D4: track 66.3 -> 65.5 mm
- net D13/SCK: track 31.8 -> 32.6 mm
- added copper zone on B.Cu, net GND
- removed copper zone on B.Cu, net (none)

Commit message: kicad v0.6
Parts:
- moved C7 0.50 mm to (194.9, 63.0)
- moved JP1 0.50 mm to (169.9, 66.0)
- moved J2 0.48 mm to (189.6, 67.0)
- moved Y1 0.45 mm to (158.4, 101.9)
- moved C6 0.38 mm to (159.7, 107.7)
- moved C5 0.31 mm to (159.7, 91.5)
Routing:
- net GND: track 214.0 -> 188.8 mm
- net +5V: track 263.3 -> 256.5 mm
- net D2: track 73.1 -> 67.6 mm
- net D12/MISO: track 28.4 -> 31.3 mm
- net A5/SCL: track 77.2 -> 79.8 mm
- net D5: track 65.4 -> 63.6 mm
- net A4/SDA: track 79.2 -> 80.1 mm
- net XTAL1: track 12.4 -> 11.7 mm
- net VCC: track 20.4 -> 19.7 mm
- net D3: track 75.5 -> 76.0 mm
- removed copper zone on F.Cu, net (none)

Commit message: kicad7
Routing:
- net +5V: track 256.5 -> 240.9 mm
- net A4/SDA: track 80.1 -> 83.7 mm
- net D11/MOSI: track 27.9 -> 31.0 mm
- net A5/SCL: track 79.8 -> 77.1 mm
- net GND: track 188.8 -> 191.5 mm
- net D10: track 30.5 -> 28.4 mm
- net D12/MISO: track 31.3 -> 29.5 mm
- net D5: track 63.6 -> 65.3 mm
- net D3: track 76.0 -> 77.5 mm
- net XTAL2: track 13.1 -> 14.1 mm
- net D4: track 65.0 -> 65.9 mm
- net D2: track 67.6 -> 68.5 mm
- net D1/Tx: track 22.2 -> 23.0 mm
- net D0/Rx: track 22.6 -> 23.4 mm
- net D6: track 58.4 -> 59.0 mm
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- added copper zone on B.Cu, net (none)
- added copper zone on F.Cu, net (none)
