File: KiCad/ardInclinometer-ATmega328/ardInclinometer-ATmega328.kicad_sch (KiCad schematic)
At the start: 26 parts, among them J1 1.8" display, SW1 Lock X, SW2 Lock Y, SW3 Lock Z, SW4 Lock all, SW5 SW_Push, U1 GY-521_MPU-6050

Commit message: new schematics and pcb
Parts:
- removed J1: 1.8" display, My_Parts:SSD1306_I2C_0.96_OLED_display_large, symbol My_Headers:4-pin_I2C_LCD_header
- added JP1: FTDI power, My_Parts:Jumper_1x02_P2.54mm_large, symbol Jumper:Jumper_2_Open
- added U2: SSD1306_I2C_display, My_Parts:SSD1306_I2C_0.96_OLED_display_large, symbol My_Parts:SSD1306_I2C_display
Connections:
- net +5V: now also JP1.2 (B), U2.2 (VCC); no longer U1.1 (VCC)
- net GND: now also U2.1 (GND)
- net A4 renamed A4/SDA
- net A4/SDA: now also U2.4 (SDA)
- net A5 renamed A5/SCL
- net A5/SCL: now also U2.3 (SCL)
- new net: JP1.1 (A), U1.1 (VCC)

Commit message: more mistakes corrected...
Parts:
- removed JP1: FTDI power, My_Parts:Jumper_1x02_P2.54mm_large, symbol Jumper:Jumper_2_Open
Connections:
- net +5V: now also U1.1 (VCC)
Changed lines of the file:
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@@
-    (stroke (width 0) (type default) (color 0 0 0 0))
-  )
-  (wire (pts (xy 220.98 39.37) (xy 220.98 46.99))
     (stroke (width 0) (type default) (color 0 0 0 0))
   )
@@
     (stroke (width 0) (type default) (color 0 0 0 0))
   )
-  (wire (pts (xy 220.98 24.13) (xy 220.98 29.21))
+  (wire (pts (xy 220.98 24.13) (xy 220.98 46.99))
     (stroke (width 0) (type default) (color 0 0 0 0))
   )
@@
     (pin "2")
   )
-  (symbol (lib_id "Jumper:Jumper_2_Open") (at 220.98 34.29 90) (unit 1)
-    (in_bom yes) (on_board yes) (fields_autoplaced)
-    (property "Reference" "JP1" (id 0) (at 222.25 33.0199 90)
-      (effects (font (size 1.27 1.27)) (justify right))
-    )
-    (property "Value" "FTDI power" (id 1) (at 222.25 35.5599 90)
-      (effects (font (size 1.27 1.27)) (justify right))
-    )
-    (property "Footprint" "My_Parts:Jumper_1x02_P2.54mm_large" (id 2) (at 220.98 34.29 0)
-      (effects (font (size 1.27 1.27)) hide)
-    )
-    (property "Datasheet" "~" (id 3) (at 220.98 34.29 0)
-      (effects (font (size 1.27 1.27)) hide)
-    )
-    (pin "1")
-    (pin "2")
-  )
   (symbol (lib_id "Device:R") (at 78.74 87.63 90) (unit 1)
     (in_bom yes) (on_board yes) (fields_autoplaced)
@@
       (reference "J2") (unit 1) (value "FTDI") (footprint "My_Headers:6-pin FTDI Programmer PinSocket large")
     )
-    (path "/48bbd05c-57f2-46d5-ae3a-a85a1af1dc7b"
-      (reference "JP1") (unit 1) (value "FTDI power") (footprint "My_Parts:Jumper_1x02_P2.54mm_large")
+    (path "/8c14ef75-6b7d-4cb1-8711-d8693b8f64e9/55052344-0687-45a9-86ac-4ca5fb142853"
+      (reference "JP1") (unit 1) (value "Power from FTDI") (footprint "My_Parts:Jumper_1x02_P2.54mm_large")
     )
     (path "/7ae86ebe-b32b-4107-b51f-cd05146b275d"

Commit message: kicad corrections and dev
Parts:
- added R11, R12: 4.7k, My_Misc:R_Axial_DIN0207_L6.3mm_D2.5mm_P10.16mm_Horizontal_large, symbol Device:R
Connections:
- net +5V: now also R11.1, R12.1
- net A4/SDA: now also R12.2
- net A5/SCL: now also R11.2
- net D11 renamed D11/MOSI
- net D12 renamed D12/MISO
- net D13 renamed D13/SCK
Other:
- moved on the sheet: U1, U2
