File: KiCad/ardInclinometer-uno/ardInclinometer-uno.kicad_sch (KiCad schematic)
At the start: 16 parts, among them U3 GY-521_MPU-6050

Commit message: kicad7
Parts:
- A1: value (none) -> Arduino_UNO_R3
- J1: value (none) -> 2-pin_power_input_header; footprint (none) -> My_Headers:2-pin_power_input_header_larger_pads
- J2: value (none) -> 4-pin_I2C_LCD_header; footprint (none) -> My_Headers:4-pin_I2C_LCD_header_larger
- R1, R2, R3, R4, R5: value (none) -> 10k; footprint (none) -> My_Misc:R_Axial_DIN0207_L6.3mm_D2.5mm_P10.16mm_Horizontal_larger_pads
- R10, R6, R7, R8, R9: value (none) -> 220R; footprint (none) -> My_Misc:R_Axial_DIN0207_L6.3mm_D2.5mm_P10.16mm_Horizontal_larger_pads
- U1: value (none) -> 6-pin_5_button_header; footprint (none) -> My_Headers:6-pin_5_switch_header_large
- U2: value (none) -> 6-pin_5_LED_header; footprint (none) -> My_Headers:6-pin_5_LED_header_large
